File: hardware/schematics/et312.sch (EAGLE design)
At the start: 52 parts, among them IC2 4066N, IC3 LM358, IC4 7809, IC5 LTC1661, IC6 7809, IC7 7805, Q1 IRL520N-H, Q2 IRL520N-H, Q3 IRF9Z24, Q4 IRL520N-H, Q5 IRL520N-H, Q6 IRF9Z24, U1 MEGA16-P, X1 HD44780LCD-1602

Commit message: Schematics
Continues Clean up
Parts:
- removed IC5: LTC1661, linear-technology:LTC2602CMS8
- added U8: LTC1661, linear-technology:LTC2602CMS8
- C1, C4: value (none) -> 470uF
- renumbered IC7 to U9
Connections:
- net GND: now also U8.GND; no longer IC5.GND
- net N$33: now also U8.VOUTB; no longer IC5.VOUTB
- net N$42: now also U8.VOUTA; no longer IC5.VOUTA
- net PB5: now also U8.SDI; no longer IC5.SDI
- net PB7: now also U8.SCK; no longer IC5.SCK
- net PD4: now also U8.!CS/LD; no longer IC5.!CS/LD
- net VCC: now also U8.REF, U8.VCC; no longer IC5.REF, IC5.VCC
Changed lines of the file:
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@@
 <part name="IC4" library="adafruit" deviceset="78*" device="T" technology="05" value="7809"/>
 <part name="GND7" library="supply1" deviceset="GND" device=""/>
-<part name="C1" library="SparkFun-Passives" deviceset="CAP_POL" device="PTH1"/>
+<part name="C1" library="SparkFun-Passives" deviceset="CAP_POL" device="PTH1" value="470uF"/>
 <part name="GND8" library="supply1" deviceset="GND" device=""/>
 <part name="C2" library="SparkFun-Passives" deviceset="CAP" device="PTH"/>
 <part name="GND9" library="supply1" deviceset="GND" device=""/>
-<part name="IC5" library="linear-technology" deviceset="LTC26*" device="MS8" technology="02C" value="LTC1661"/>
+<part name="U8" library="linear-technology" deviceset="LTC26*" device="MS8" technology="02C" value="LTC1661"/>
 <part name="P+1" library="supply1" deviceset="VCC" device="" value="+5V"/>
-<part name="P+2" library="supply1" deviceset="VCC" device="" value="+5V"/>
 <part name="R6" library="eagle-ltspice" deviceset="R" device="0207/10" value="100k"/>
 <part name="R7" library="eagle-ltspice" deviceset="R" device="0207/10" value="100k"/>
@@
 <part name="IC6" library="adafruit" deviceset="78*" device="T" technology="05" value="7809"/>
 <part name="GND18" library="supply1" deviceset="GND" device=""/>
-<part name="C4" library="SparkFun-Passives" deviceset="CAP_POL" device="PTH1"/>
+<part name="C4" library="SparkFun-Passives" deviceset="CAP_POL" device="PTH1" value="470uF"/>
 <part name="GND19" library="supply1" deviceset="GND" device=""/>
 <part name="P+11" library="supply1" deviceset="VCC" device="" value="+9V 1"/>
-<part name="IC7" library="adafruit" deviceset="78*" device="T" technology="05" value="7805"/>
+<part name="U9" library="adafruit" deviceset="78*" device="T" technology="05" value="7805"/>
 <part name="GND20" library="supply1" deviceset="GND" device=""/>
 <part name="R22" library="eagle-ltspice" deviceset="R" device="0207/10" value="100k"/>
@@
 <part name="SUPPLY6" library="SparkFun-Aesthetics" deviceset="5V" device=""/>
 <part name="SUPPLY7" library="SparkFun-Aesthetics" deviceset="5V" device=""/>
+<part name="P+10" library="supply1" deviceset="VCC" device="" value="+5V"/>
 </parts>
 <sheets>
@@
 <instance part="GND19" gate="1" x="40.64" y="53.34"/>
 <instance part="P+11" gate="VCC" x="48.26" y="73.66"/>
-<instance part="IC7" gate="A1" x="68.58" y="71.12"/>
+<instance part="U9" gate="A1" x="68.58" y="71.12"/>
 <instance part="GND20" gate="1" x="68.58" y="58.42"/>
 <instance part="SUPPLY7" gate="G$1" x="86.36" y="73.66"/>
@@
 <segment>
 <pinref part="GND20" gate="1" pin="GND"/>
-<pinref part="IC7" gate="A1" pin="GND"/>
+<pinref part="U9" gate="A1" pin="GND"/>
 <wire x1="68.58" y1="60.96" x2="68.58" y2="63.5" width="0.1524" layer="91"/>
 </segment>
@@
 </segment>
 <segment>
-<pinref part="IC7" gate="A1" pin="VO"/>
+<pinref part="U9" gate="A1" pin="VO"/>
 <wire x1="78.74" y1="71.12" x2="86.36" y2="71.12" width="0.1524" layer="91"/>
 <pinref part="SUPPLY7" gate="G$1" pin="5V"/>
@@
 <instance part="C2" gate="G$1" x="182.88" y="129.54"/>
 <instance part="GND9" gate="1" x="149.86" y="129.54"/>
-<instance part="IC5" gate="-1" x="81.28" y="147.32"/>
-<instance part="P+1" gate="VCC" x="66.04" y="165.1"/>
-<instance part="P+2" gate="VCC" x="99.06" y="147.32"/>
+<instance part="U8" gate="-1" x="71.12" y="132.08"/>
+<instance part="P+1" gate="VCC" x="55.88" y="149.86"/>
 <instance part="R6" gate="G$1" x="149.86" y="157.48"/>
 <instance part="R7" gate="G$1" x="127" y="132.08" rot="R90"/>
@@
 <instance part="R21" gate="G$1" x="152.4" y="20.32" rot="R90"/>
 <instance part="GND15" gate="1" x="152.4" y="10.16"/>
-<instance part="GND16" gate="1" x="66.04" y="127"/>
+<instance part="GND16" gate="1" x="55.88" y="111.76"/>
 <instance part="R22" gate="G$1" x="116.84" y="53.34"/>
 <instance part="P+13" gate="VCC" x="149.86" y="152.4"/>
@@
 <instance part="SUPPLY6" gate="G$1" x="243.84" y="157.48"/>
 <instance part="FRAME6" gate="G$1" x="0" y="0"/>
+<instance part="P+10" gate="VCC" x="88.9" y="149.86"/>
 </instances>
 <busses>
@@
 </segment>
 <segment>
+<pinref part="U8" gate="-1" pin="GND"/>
+<wire x1="58.42" y1="124.46" x2="55.88" y2="124.46" width="0.1524" layer="91"/>
 <pinref part="GND16" gate="1" pin="GND"/>
-<pinref part="IC5" gate="-1" pin="GND"/>
-<wire x1="66.04" y1="129.54" x2="68.58" y2="139.7" width="0.1524" layer="91"/>
+<wire x1="55.88" y1="124.46" x2="55.88" y2="114.3" width="0.1524" layer="91"/>
 </segment>
 </net>
@@
 </net>
 <net name="VCC" class="0">
-<segment>
-<pinref part="IC5" gate="-1" pin="REF"/>
-<wire x1="93.98" y1="144.78" x2="99.06" y2="144.78" width="0.1524" layer="91"/>
-<pinref part="P+2" gate="VCC" pin="VCC"/>
-</segment>
 <segment>
 <pinref part="R9" gate="G$1" pin="2"/>
@@
 </segment>
 <segment>
-<pinref part="IC5" gate="-1" pin="VCC"/>
-<pinref part="P+1" gate="VCC" pin="VCC"/>
-<wire x1="68.58" y1="154.94" x2="66.04" y2="162.56" width="0.1524" layer="91"/>
-</segment>
-<segment>
 <pinref part="P+7" gate="VCC" pin="VCC"/>
 <wire x1="175.26" y1="40.64" x2="175.26" y2="38.1" width="0.1524" layer="91"/>
@@
 <pinref part="P+13" gate="VCC" pin="VCC"/>
 </segment>
+<segment>
+<pinref part="P+1" gate="VCC" pin="VCC"/>
+<wire x1="55.88" y1="147.32" x2="55.88" y2="139.7" width="0.1524" layer="91"/>
+<pinref part="U8" gate="-1" pin="VCC"/>
+<wire x1="55.88" y1="139.7" x2="58.42" y2="139.7" width="0.1524" layer="91"/>
+</segment>
+<segment>
+<pinref part="U8" gate="-1" pin="REF"/>
+<pinref part="P+10" gate="VCC" pin="VCC"/>
+<wire x1="83.82" y1="129.54" x2="88.9" y2="129.54" width="0.1524" layer="91"/>
+<wire x1="88.9" y1="129.54" x2="88.9" y2="147.32" width="0.1524" layer="91"/>
+</segment>
 </net>
 <net name="N$22" class="0">
@@
 <net name="PB7" class="0">
 <segment>
-<wire x1="55.88" y1="144.78" x2="68.58" y2="144.78" width="0.1524" layer="91"/>
-<pinref part="IC5" gate="-1" pin="SCK"/>
-<label x="55.88" y="144.78" size="1.778" layer="95" rot="R180" xref="yes"/>
+<wire x1="45.72" y1="129.54" x2="58.42" y2="129.54" width="0.1524" layer="91"/>
+<pinref part="U8" gate="-1" pin="SCK"/>
+<label x="45.72" y="129.54" size="1.778" layer="95" rot="R180" xref="yes"/>
 </segment>
 </net>
 <net name="PD4" class="0">
 <segment>
-<pinref part="IC5" gate="-1" pin="!CS/LD"/>
-<wire x1="55.88" y1="149.86" x2="68.58" y2="149.86" width="0.1524" layer="91"/>
-<label x="55.88" y="149.86" size="1.778" layer="95" rot="R180" xref="yes"/>
+<pinref part="U8" gate="-1" pin="!CS/LD"/>
+<wire x1="45.72" y1="134.62" x2="58.42" y2="134.62" width="0.1524" layer="91"/>
+<label x="45.72" y="134.62" size="1.778" layer="95" rot="R180" xref="yes"/>
 </segment>
 </net>
@@
 <net name="N$33" class="0">
 <segment>
-<pinref part="IC5" gate="-1" pin="VOUTB"/>
+<pinref part="U8" gate="-1" pin="VOUTB"/>
 <pinref part="R22" gate="G$1" pin="1"/>
-<wire x1="111.76" y1="53.34" x2="104.14" y2="53.34" width="0.1524" layer="91"/>
-<wire x1="104.14" y1="53.34" x2="104.14" y2="149.86" width="0.1524" layer="91"/>
-<wire x1="104.14" y1="149.86" x2="93.98" y2="149.86" width="0.1524" layer="91"/>
+<wire x1="111.76" y1="53.34" x2="93.98" y2="53.34" width="0.1524" layer="91"/>
+<wire x1="93.98" y1="53.34" x2="93.98" y2="134.62" width="0.1524" layer="91"/>
+<wire x1="93.98" y1="134.62" x2="83.82" y2="134.62" width="0.1524" layer="91"/>
 </segment>
 </net>
@@
 <segment>
 <pinref part="R11" gate="G$1" pin="1"/>
-<wire x1="111.76" y1="139.7" x2="106.68" y2="139.7" width="0.1524" layer="91"/>
-<wire x1="106.68" y1="139.7" x2="106.68" y2="154.94" width="0.1524" layer="91"/>
-<pinref part="IC5" gate="-1" pin="VOUTA"/>
-<wire x1="106.68" y1="154.94" x2="93.98" y2="154.94" width="0.1524" layer="91"/>
+<pinref part="U8" gate="-1" pin="VOUTA"/>
+<wire x1="111.76" y1="139.7" x2="83.82" y2="139.7" width="0.1524" layer="91"/>
 </segment>
 </net>
 <net name="PB5" class="0">
 <segment>
-<pinref part="IC5" gate="-1" pin="SDI"/>
-<wire x1="93.98" y1="139.7" x2="99.06" y2="139.7" width="0.1524" layer="91"/>
-<wire x1="99.06" y1="139.7" x2="99.06" y2="132.08" width="0.1524" layer="91"/>
-<wire x1="99.06" y1="132.08" x2="55.88" y2="132.08" width="0.1524" layer="91"/>
-<label x="55.88" y="132.08" size="1.778" layer="95" rot="R180" xref="yes"/>
-</segment>
-</net>
+<pinref part="U8" gate="-1" pin="SDI"/>
+<wire x1="83.82" y1="124.46" x2="88.9" y2="124.46" width="0.1524" layer="91"/>
+<wire x1="88.9" y1="124.46" x2="88.9" y2="116.84" width="0.1524" layer="91"/>
+<wire x1="88.9" y1="116.84" x2="45.72" y2="116.84" width="0.1524" layer="91"/>
+<label x="45.72" y="116.84" size="1.778" layer="95" rot="R180" xref="yes"/>
+</segment>
+</net>

Commit message: Schematics
WIP
Connections:
- new net N$16: 10WAY_RIBBON1.10
- new net N$17: IC4.VI, IC6.VI, U9.VI
- new net N$6: 10WAY_RIBBON1.4
- new net N$9: 10WAY_RIBBON1.9
Other:
- moved on the sheet: U9

Commit message: schemtaics
wip
Parts:
- added RP5A, RP5B: 390, rcl:R-EU_0207/7
Connections:
- new net N$23: LED2.A, RP5B.1
- new net N$29: LED1.A, RP5A.1
- net 5V: now also RP5A.2, RP5B.2
- net PD5: now also LED2.C
- net PD6: now also LED1.C
Other:
- moved on the sheet: IC2A, IC2B, LED1, LED2
Changed lines of the file:
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@@
 <part name="GND7" library="SparkFun-Aesthetics" deviceset="GND" device=""/>
 <part name="GND8" library="SparkFun-Aesthetics" deviceset="GND" device=""/>
+<part name="RP5A" library="rcl" deviceset="R-EU_" device="0207/7" value="390"/>
+<part name="RP5B" library="rcl" deviceset="R-EU_" device="0207/7" value="390"/>
+<part name="SUPPLY8" library="SparkFun-Aesthetics" deviceset="5V" device=""/>
 </parts>
 <sheets>
@@
 <instance part="SUPPLY5" gate="G$1" x="99.06" y="149.86"/>
 <instance part="J2" gate="A" x="50.8" y="137.16"/>
-<instance part="LED1" gate="G$1" x="205.74" y="71.12"/>
-<instance part="LED2" gate="G$1" x="215.9" y="71.12"/>
+<instance part="LED1" gate="G$1" x="210.82" y="86.36"/>
+<instance part="LED2" gate="G$1" x="220.98" y="86.36"/>
 <instance part="GND4" gate="1" x="210.82" y="43.18"/>
 <instance part="IC4" gate="A1" x="27.94" y="38.1"/>
@@
 <instance part="GND7" gate="1" x="40.64" y="53.34"/>
 <instance part="GND8" gate="1" x="40.64" y="88.9"/>
+<instance part="RP5A" gate="G$1" x="210.82" y="96.52" rot="R90"/>
+<instance part="RP5B" gate="G$1" x="220.98" y="96.52" rot="R90"/>
+<instance part="SUPPLY8" gate="G$1" x="210.82" y="106.68"/>
 </instances>
 <busses>
@@
 <wire x1="48.26" y1="99.06" x2="48.26" y2="104.14" width="0.1524" layer="91"/>
 </segment>
+<segment>
+<pinref part="SUPPLY8" gate="G$1" pin="5V"/>
+<pinref part="RP5A" gate="G$1" pin="2"/>
+<wire x1="210.82" y1="106.68" x2="210.82" y2="104.14" width="0.1524" layer="91"/>
+<wire x1="210.82" y1="104.14" x2="210.82" y2="101.6" width="0.1524" layer="91"/>
+<wire x1="210.82" y1="104.14" x2="220.98" y2="104.14" width="0.1524" layer="91"/>
+<wire x1="220.98" y1="104.14" x2="220.98" y2="101.6" width="0.1524" layer="91"/>
+<pinref part="RP5B" gate="G$1" pin="2"/>
+<junction x="210.82" y="104.14"/>
+</segment>
 </net>
 <net name="JTAG7" class="0">
@@
 <segment>
 <pinref part="U1" gate="G$1" pin="(OC1A)PD5"/>
-<wire x1="147.32" y1="71.12" x2="157.48" y2="71.12" width="0.1524" layer="91"/>
-<label x="157.48" y="71.12" size="1.778" layer="95" xref="yes"/>
+<pinref part="LED2" gate="G$1" pin="C"/>
+<wire x1="147.32" y1="71.12" x2="220.98" y2="71.12" width="0.1524" layer="91"/>
+<wire x1="220.98" y1="71.12" x2="220.98" y2="81.28" width="0.1524" layer="91"/>
 </segment>
 </net>
@@
 <segment>
 <pinref part="U1" gate="G$1" pin="(ICP)PD6"/>
-<wire x1="147.32" y1="73.66" x2="157.48" y2="73.66" width="0.1524" layer="91"/>
-<label x="157.48" y="73.66" size="1.778" layer="95" xref="yes"/>
+<pinref part="LED1" gate="G$1" pin="C"/>
+<wire x1="147.32" y1="73.66" x2="210.82" y2="73.66" width="0.1524" layer="91"/>
+<wire x1="210.82" y1="73.66" x2="210.82" y2="81.28" width="0.1524" layer="91"/>
 </segment>
 </net>
@@
 </segment>
 </net>
+<net name="N$23" class="0">
+<segment>
+<pinref part="RP5B" gate="G$1" pin="1"/>
+<pinref part="LED2" gate="G$1" pin="A"/>
+<wire x1="220.98" y1="91.44" x2="220.98" y2="88.9" width="0.1524" layer="91"/>
+</segment>
+</net>
+<net name="N$29" class="0">
+<segment>
+<pinref part="RP5A" gate="G$1" pin="1"/>
+<pinref part="LED1" gate="G$1" pin="A"/>
+<wire x1="210.82" y1="91.44" x2="210.82" y2="88.9" width="0.1524" layer="91"/>
+</segment>
+</net>
 </nets>
 </sheet>
@@
 <instances>
 <instance part="FRAME4" gate="G$1" x="0" y="0"/>
-<instance part="IC2" gate="A" x="83.82" y="139.7" smashed="yes">
-<attribute name="NAME" x="76.2" y="145.415" size="1.778" layer="95"/>
-<attribute name="VALUE" x="76.2" y="132.08" size="1.778" layer="96"/>
+<instance part="IC2" gate="A" x="175.26" y="144.78" smashed="yes">
+<attribute name="NAME" x="167.64" y="150.495" size="1.778" layer="95"/>
+<attribute name="VALUE" x="167.64" y="137.16" size="1.778" layer="96"/>
 </instance>
-<instance part="IC2" gate="B" x="175.26" y="139.7"/>
+<instance part="IC2" gate="B" x="83.82" y="144.78"/>
 <instance part="IC2" gate="C" x="83.82" y="96.52"/>
 <instance part="IC2" gate="D" x="175.26" y="96.52"/>
@@
 <segment>
 <pinref part="IC2" gate="A" pin="C"/>
-<wire x1="71.12" y1="137.16" x2="68.58" y2="137.16" width="0.1524" layer="91"/>
-<label x="68.58" y="137.16" size="1.778" layer="95" rot="R180" xref="yes"/>
+<wire x1="162.56" y1="142.24" x2="160.02" y2="142.24" width="0.1524" layer="91"/>
+<label x="160.02" y="142.24" size="1.778" layer="95" rot="R180" xref="yes"/>
 </segment>
 <segment>
@@
 <segment>
 <pinref part="IC2" gate="B" pin="C"/>
-<wire x1="160.02" y1="137.16" x2="162.56" y2="137.16" width="0.1524" layer="91"/>
-<label x="160.02" y="137.16" size="1.778" layer="95" rot="R180" xref="yes"/>
+<wire x1="68.58" y1="142.24" x2="71.12" y2="142.24" width="0.1524" layer="91"/>
+<label x="68.58" y="142.24" size="1.778" layer="95" rot="R180" xref="yes"/>
 </segment>
 <segment>
@@
 <segment>
 <pinref part="IC2" gate="A" pin="B"/>
-<wire x1="96.52" y1="142.24" x2="99.06" y2="142.24" width="0.1524" layer="91"/>
-<label x="99.06" y="142.24" size="1.778" layer="95" xref="yes"/>
+<wire x1="187.96" y1="147.32" x2="190.5" y2="147.32" width="0.1524" layer="91"/>
+<label x="190.5" y="147.32" size="1.778" layer="95" xref="yes"/>
 </segment>
 </net>
@@
 <segment>
 <pinref part="IC2" gate="B" pin="B"/>
-<wire x1="187.96" y1="142.24" x2="190.5" y2="142.24" width="0.1524" layer="91"/>
-<label x="190.5" y="142.24" size="1.778" layer="95" xref="yes"/>
+<wire x1="96.52" y1="147.32" x2="99.06" y2="147.32" width="0.1524" layer="91"/>
+<label x="99.06" y="147.32" size="1.778" layer="95" xref="yes"/>
 </segment>
 </net>
@@
 <pinref part="10WAY_RIBBON1" gate="G$1" pin="1"/>
 <wire x1="17.78" y1="137.16" x2="48.26" y2="137.16" width="0.1524" layer="91"/>
-<wire x1="48.26" y1="137.16" x2="48.26" y2="149.86" width="0.1524" layer="91"/>
-<wire x1="48.26" y1="149.86" x2="160.02" y2="149.86" width="0.1524" layer="91"/>
-<wire x1="160.02" y1="149.86" x2="160.02" y2="142.24" width="0.1524" layer="91"/>
+<wire x1="48.26" y1="137.16" x2="48.26" y2="147.32" width="0.1524" layer="91"/>
+<wire x1="48.26" y1="147.32" x2="71.12" y2="147.32" width="0.1524" layer="91"/>
 <pinref part="IC2" gate="B" pin="A"/>
-<wire x1="160.02" y1="142.24" x2="162.56" y2="142.24" width="0.1524" layer="91"/>
 </segment>
 </net>
 <net name="N$8" class="0">
 <segment>
-<pinref part="IC2" gate="A" pin="A"/>
-<wire x1="71.12" y1="142.24" x2="45.72" y2="142.24" width="0.1524" layer="91"/>
-<wire x1="45.72" y1="142.24" x2="45.72" y2="139.7" width="0.1524" layer="91"/>
+<wire x1="45.72" y1="154.94" x2="45.72" y2="139.7" width="0.1524" layer="91"/>
 <pinref part="10WAY_RIBBON1" gate="G$1" pin="2"/>
 <wire x1="45.72" y1="139.7" x2="17.78" y2="139.7" width="0.1524" layer="91"/>
-</segment>
-</net>
+<wire x1="45.72" y1="154.94" x2="160.02" y2="154.94" width="0.1524" layer="91"/>
+<wire x1="160.02" y1="154.94" x2="160.02" y2="147.32" width="0.1524" layer="91"/>
+<pinref part="IC2" gate="A" pin="A"/>
+<wire x1="160.02" y1="147.32" x2="162.56" y2="147.32" width="0.1524" layer="91"/>
+</segment>
+</net>
