File: hardware/schematics/et312.sch (EAGLE design)
At the start: 54 parts, among them IC2 4066N, IC3 LM358, IC4 7809, IC6 7809, Q1 IRL520N-H, Q2 IRL520N-H, Q3 IRF9Z24, Q4 IRL520N-H, Q5 IRL520N-H, Q6 IRF9Z24, U1 MEGA16-P, U8 LTC1661, U9 7805, X1 HD44780LCD-1602

Commit message: Schematics
more wip
Changed lines of the file:
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@@
 <part name="RP5B" library="rcl" deviceset="R-EU_" device="0207/7" value="390"/>
 <part name="SUPPLY8" library="SparkFun-Aesthetics" deviceset="5V" device=""/>
+<part name="GND18" library="SparkFun-Aesthetics" deviceset="GND" device=""/>
+<part name="SUPPLY9" library="SparkFun-Aesthetics" deviceset="5V" device=""/>
 </parts>
 <sheets>
@@
 <instance part="FRAME5" gate="G$1" x="0" y="0"/>
 <instance part="X1" gate="G$1" x="119.38" y="88.9"/>
+<instance part="GND18" gate="1" x="165.1" y="111.76"/>
+<instance part="SUPPLY9" gate="G$1" x="165.1" y="119.38"/>
 </instances>
 <busses>

Commit message: Updates to schematics, based on hand drawn schematics
Parts:
- removed U8: LTC1661, linear-technology:LTC2602CMS8
- added C10, C15, C16, C9: 100n, rcl:C-EU050-025X075
- added C11: 1u, rcl:C-EU050-025X075
- added C12, C13, C14: 1u, rcl:CPOL-EUE2.5-5
- added C5: (no value), rcl:CPOL-EUE2.5-6
- added C6, C7: (no value), rcl:CPOL-EUE3.5-10
- added C8: (no value), rcl:C-EU050-025X075
- added D1: 1N4004, diode:1N4004
- added D2, D3: 1N4004, adafruit:1N4004
- added IC1: LM324N, linear:LM324N
- added IC5: LM358N, linear:LM358N
- added J1: BATTERY_CONNDEANS, SparkFun-Connectors:BATTERY_CONNDEANS
- added JP1: POWER_JACKSLT, SparkFun-Connectors:POWER_JACKSLT
- added L1: (no value), rcl:L-EU0207/10
- added Q7: 2N3906, transistor-pnp:2N3906
- added QF1: 16M20AUM1, crystal:16M20AUM1
- added R23, R24: (no value), rcl:R-EU_0207/10
- added R25: (no value), pot:TRIM_EU-LI10
- added R26, R29: 390R, rcl:R-EU_0207/10
- added R27, R28, R31, R35, R41, R44, R45, R48: 100K, rcl:R-EU_0207/10
- added R30: 10K, rcl:R-EU_0207/10
- added R32, R36, R38, R43, R51: 20K, rcl:R-EU_0207/10
- added R33, R34, R46, R47, R49: 4.7K, rcl:R-EU_0207/10
- added R37, R39, R42, R50: 1M, rcl:R-EU_0207/10
- added R40: 10K, rcl:R-EU_0207/7
- added R52: 0.5R, eagle-ltspice:R0207/10
- added RP1: 20K, rcl:R-EU_0207/7
- added RP5B1: 47, rcl:R-EU_0207/7
- added RP6: 100K, rcl:R-EU_0207/7
- added RP7: 3.3K, rcl:R-EU_0207/7
- added T1: 2N3904, transistor:2N3904
- added T2, T3: (no value), Eagle_POWER_MAGNETICS_rev16b:WE-FB_LT35XX/LT3748_EFD25_750310988
- added U$1: LM2941, JAEB:LM2941
- added U$2: MAX548, JAEB:MAX548
- added X2, X3, X4, X5, X6: STEREOJACK, adafruit:STEREOJACK
Connections:
- removed net N$16: 10WAY_RIBBON1.10
- removed net N$6: 10WAY_RIBBON1.4
- removed net PA2: U1.(ADC2)PA2
- removed net PA3: U1.(ADC3)PA3
- removed net PA6: U1.(ADC6)PA6
- removed net PA7: U1.(ADC7)PA7
- removed net PB4: U1.(SS)PB4
- removed net PB5: U1.(MOSI)PB5, U8.SDI
- removed net PB6: U1.(MISO)PB6
- removed net PB7: U1.(SCK)PB7, U8.SCK
- removed net PD4: U1.(OC1B)PD4, U8.!CS/LD
- new net !CS: U$2.!CS, U1.(OC1B)PD4
- new net +12V: C7.+, C8.1, D1.C, IC4.VI, IC6.VI, J2.2, L1.2, R40.2, U9.VI
- new net +5V: Q7.E, R28.1, R35.2, R42.2, R47.2
- new net +9V1: C2.2, C4.+, IC6.VO, Q3.S, R8.2
- new net +9V2: C1.+, C3.2, IC4.VO, Q6.S, R18.2
- new net N$30: R25.S, X1.VO
- new net N$31: J1.+, L1.1
- new net N$32: QF1.1, U1.XTAL2
- new net N$43: R23.1, R24.2, U$1.ADJ
- new net N$44: R29.2, R30.1, X4.5
- new net N$45: C6.+, D1.A, R23.2, U$1.OUT
- new net N$46: R27.2, X4.2
- new net N$47: RP5B1.1, X1.A
- new net N$48: R27.1, T1.B
- new net N$51: R31.2, R32.1
- new net N$52: Q7.C, R29.1
- new net N$53: IC1A.-IN, R36.1, R37.1
- new net N$54: D2.A, IC1A.OUT, IC1D.+IN, R37.2
- new net N$55: R33.1, X3.2
- new net N$56: R34.1, X3.5
- new net N$57: C9.1, R34.2
- new net N$60: IC1B.-IN, R38.2, R39.1
- new net N$61: IC5B.OUT
- new net N$62: IC1C.-IN, IC1D.-IN, R41.1, R42.1
- new net N$63: C10.2, IC1B.+IN, R43.2
- new net N$66: T3.3, X6.1
- new net N$67: T3.2, X6.2, X6.5
- new net N$69: D3.A, IC1B.OUT, IC1C.+IN, R39.2
- new net N$71: R46.1, X2.2, X2.5
- new net N$72: C14.+, C15.1, R46.2, R47.1
- new net N$73: C15.2, IC5A.+IN, R48.2
- new net N$74: IC5A.-IN, R50.1, R51.2
- new net N$75: IC5A.OUT, IC5B.-IN, R49.2, R50.2
- new net N$76: C16.1, R49.1
- new net N$77: T2.3, X5.1
- new net N$78: T2.2, X5.2, X5.5
- new net PA6_AINB: C12.+, D2.C, R44.1, U1.(ADC6)PA6
- new net PA7_AINA: C13.+, D3.C, R45.1, U1.(ADC7)PA7
- new net RB10: 10WAY_RIBBON1.10, C9.2, R35.1
- new net RB4: 10WAY_RIBBON1.4, IC1A.+IN
- new net RB9: 10WAY_RIBBON1.9, C16.2, R33.2
- new net V+: C5.+, JP1.PWR, RP6.2, U$1.IN
- net 5V: now also J2.14, R25.E, RP5B1.2, X1.VDD
- net GND: now also C11.1, C12.-, C13.-, C14.-, C5.-, C6.-, C7.-, C8.2, IC5B.+IN, J1.-, J2.10, J2.12, JP1.GND, JP1.GNDBREAK, R24.1, R25.A, R26.1, R30.2, R32.2, R36.2, R38.1, R41.2, R43.1, R44.2, R45.2, R48.1, R51.1, R52.1, RP1.1, RP7.1, T1.E, U$1.!ON, U$1.GND, U$2.GND, X1.VSS, X2.1, X3.1; no longer U8.GND
- net JTAG11: now also U1.(MISO)PB6
- net JTAG13: now also U$2.SCLK, U1.(SCK)PB7
- net JTAG7: now also U1.(SS)PB4
- net JTAG9: now also U$2.DIN, U1.(MOSI)PB5
- net N$17: now also QF1.3, U1.XTAL1; no longer IC4.VI, IC6.VI, U9.VI
- net N$33: now also U$2.OUTA; no longer U8.VOUTB
- net N$34: now also T2.1
- net N$35: now also T2.5
- net N$36: now also T3.1
- net N$37: now also T3.5
- net N$38: now also T3.4
- net N$39: now also T2.4
- net N$42: now also U$2.OUTB; no longer U8.VOUTA
- net N$9: now also R26.2, X4.1; no longer 10WAY_RIBBON1.9
- net PA0: now also R52.2
- net PA1: now also C10.1, C11.2
- net PA4: now also R40.1, RP7.2, U1.(ADC3)PA3
- net PA5: now also RP1.2, RP6.1, U1.(ADC2)PA2
- net PB0: now also R12.2, R13.1; no longer R14.1, R21.2
- net PB1: now also R14.1, R21.2; no longer R12.2, R13.1
- net PB2: now also R1.2, R2.1; no longer R3.1, R4.2
- net PB3: now also R3.1, R4.2; no longer R1.2, R2.1
- net PD0: now also R28.2, T1.C
- net PD1: now also Q7.B, R31.1
- net PD2: now also IC1D.OUT
- net PD3: now also IC1C.OUT
- net PD7: now also X1.K
- net VCC: now also U$2.!LDAC, U$2.VDD; no longer C1.+, C2.2, C3.2, C4.+, IC4.VO, IC6.VO, Q3.S, Q6.S, R18.2, R8.2, U8.REF, U8.VCC
Other:
- note added: "Possible transformer: Wurth 750811048"
- note added: "This connector isn't fully connected yet!"
